File: routage/routage.kicad_sch (KiCad schematic)
At the start: 51 parts, among them J2 Conn_01x02, J3 Conn_01x03, Q1 2N2907, Q10 TIP32, Q11 BD138, Q12 TIP31, Q13 2N2222, Q2 2N2907, Q3 2N2907, Q4 2N2222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

Commit message: placement corrigé
Parts:
- removed Q8: BD139, Package_TO_SOT_THT:TO-126-3_Vertical, symbol Device:Q_NPN_CEB
- added Q8: BD139, symbol Device:Q_NPN_ECB
Connections:
- net at Q6.3 (C), Q9.3 (B), RV1.1: now also Q8.2 (C)
- net at C2.2, Q11.3 (B), Q4.3 (C)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: now also Q8.1 (E)
- net at RV1.2: now also Q8.3 (B)
Changed lines of the file:
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@@
     (pin "1")
-  )
-  (symbol (lib_id "Device:Q_NPN_CEB") (at 127 67.31 0) (unit 1)
-    (in_bom yes) (on_board yes) (fields_autoplaced)
-    (property "Reference" "Q8" (id 0) (at 132.08 66.0399 0)
-      (effects (font (size 1.27 1.27)) (justify left))
-    )
-    (property "Value" "BD139" (id 1) (at 132.08 68.5799 0)
-      (effects (font (size 1.27 1.27)) (justify left))
-    )
-    (property "Footprint" "Package_TO_SOT_THT:TO-126-3_Vertical" (id 2) (at 132.08 64.77 0)
-      (effects (font (size 1.27 1.27)) hide)
-    )
-    (property "Datasheet" "~" (id 3) (at 127 67.31 0)
-      (effects (font (size 1.27 1.27)) hide)
-    )
-    (pin "1")
-    (pin "2")
-    (pin "3")
   )
   (symbol (lib_id "power:PWR_FLAG") (at 60.96 186.69 180) (unit 1)
@@
     )
     (pin "1")
+  )
+  (symbol (lib_id "Device:Q_NPN_ECB") (at 127 67.31 0) (unit 1)
+    (in_bom yes) (on_board yes) (fields_autoplaced)
+    (property "Reference" "Q8" (id 0) (at 132.08 66.0399 0)
+      (effects (font (size 1.27 1.27)) (justify left))
+    )
+    (property "Value" "BD139" (id 1) (at 132.08 68.5799 0)
+      (effects (font (size 1.27 1.27)) (justify left))
+    )
+    (property "Footprint" "" (id 2) (at 132.08 64.77 0)
+      (effects (font (size 1.27 1.27)) hide)
+    )
+    (property "Datasheet" "~" (id 3) (at 127 67.31 0)
+      (effects (font (size 1.27 1.27)) hide)
+    )
+    (pin "1")
+    (pin "2")
+    (pin "3")
   )
   (symbol (lib_id "Device:Q_NPN_EBC") (at 222.25 100.33 0) (mirror y) (unit 1)
@@
       (reference "Q7") (unit 1) (value "2N2907") (footprint "Package_TO_SOT_THT:TO-18-3")
     )
-    (path "/16e0cb01-317c-4e81-8ff0-3c8916eae187"
-      (reference "Q8") (unit 1) (value "BD139") (footprint "Package_TO_SOT_THT:TO-126-3_Vertical")
+    (path "/b5ea958d-0cfd-4df9-ac20-3edbdc47b6ee"
+      (reference "Q8") (unit 1) (value "BD139") (footprint "")
     )
     (path "/f2a39f2f-d34c-4216-b5ae-8ee0bee406d3"
